Commit message: update submodule code

File: robots/hands/omni_hand/omnihand_right.urdf (robot description, URDF)
Before this commit: robot omnihand, 24 links, 23 joints
Links:
- link R_index_abad: geometry visual mesh filename=meshes/finger_abad.STL
- link R_index_dip: geometry collision cylinder length=0.034 radius=0.007; visual mesh filename=meshes/finger_dip.STL
- link R_index_pip: geometry collision cylinder length=0.044 radius=0.01; visual mesh filename=meshes/finger_pip.STL
- link R_middle_abad: geometry visual mesh filename=meshes/finger_abad.STL
- link R_middle_dip: geometry collision cylinder length=0.034 radius=0.007; visual mesh filename=meshes/finger_dip.STL
- link R_middle_pip: geometry collision cylinder length=0.044 radius=0.01; visual mesh filename=meshes/finger_pip.STL
- link R_palm: geometry collision box size=0.04 0.082 0.085; collision cylinder length=0.0145 radius=0.028
- link R_pinky_abad: geometry visual mesh filename=meshes/finger_abad.STL
- link R_pinky_dip: geometry collision cylinder length=0.034 radius=0.007; visual mesh filename=meshes/finger_dip.STL
- link R_pinky_pip: geometry collision cylinder length=0.044 radius=0.01; visual mesh filename=meshes/finger_pip.STL
- link R_ring_abad: geometry visual mesh filename=meshes/finger_abad.STL
- link R_ring_dip: geometry collision cylinder length=0.034 radius=0.007; visual mesh filename=meshes/finger_dip.STL
- link R_ring_pip: geometry collision cylinder length=0.044 radius=0.01; visual mesh filename=meshes/finger_pip.STL
- link R_thumb_abad: geometry visual mesh filename=meshes/thumb_abad.STL
- link R_thumb_dip: geometry collision cylinder length=0.023 radius=0.011; visual mesh filename=meshes/thumb_dip.STL
- link R_thumb_mcp: geometry collision box size=0.029 0.042 0.0325; visual mesh filename=meshes/thumb_mcp.STL
- link R_thumb_pip: geometry collision box size=0.019 0.035 0.0225; visual mesh filename=meshes/thumb_pip.STL
- link R_thumb_roll: geometry visual mesh filename=meshes/r_thumb_roll.STL

Commit message: update submodule code

File: robots/hands/omni_hand/omnihand_right.urdf (robot description, URDF)
Before this commit: robot omnihand, 24 links, 23 joints
Joints:
- joint R_index_dip_joint: mimic joint=R_index_pip_joint multiplier=1.097 offset=0 -> joint=R_index_pip_joint multiplier=0.3 offset=0
- joint R_middle_dip_joint: mimic joint=R_middle_pip_joint multiplier=1.097 offset=0 -> joint=R_middle_pip_joint multiplier=0.3 offset=0
- joint R_pinky_dip_joint: mimic joint=R_pinky_pip_joint multiplier=1.097 offset=0 -> joint=R_pinky_pip_joint multiplier=0.3 offset=0
- joint R_ring_dip_joint: mimic joint=R_ring_pip_joint multiplier=1.097 offset=0 -> joint=R_ring_pip_joint multiplier=0.3 offset=0
- joint R_thumb_dip_joint: mimic joint=R_thumb_mcp_joint multiplier=1.3 offset=0 -> joint=R_thumb_mcp_joint multiplier=0.5 offset=0
- joint R_thumb_pip_joint: mimic joint=R_thumb_mcp_joint multiplier=1.33 offset=0 -> joint=R_thumb_mcp_joint multiplier=0.5 offset=0

File: robots/hands/omnipro_hand/omniprohand_right.urdf (robot description, URDF)
Before this commit: robot omniprohand, 25 links, 24 joints
Joints:
- joint thumb_cmc_yaw: limit lower=0 upper=0.3 effort=100 velocity=1 -> lower=0 upper=1.3868 effort=100 velocity=1
- joint thumb_ip: limit lower=0 upper=0.1 effort=100 velocity=1 -> lower=0 upper=0.3781 effort=100 velocity=1
- joint thumb_mcp: limit lower=0 upper=0.8 effort=100 velocity=1 -> lower=0 upper=0.2908 effort=100 velocity=1

Commit message: update submodule code

File: robots/hands/omni_hand/omnihand_right.urdf (robot description, URDF)
Before this commit: robot omnihand, 24 links, 23 joints
Joints:
- joint R_index_dip_joint: mimic joint=R_index_pip_joint multiplier=0.3 offset=0 -> joint=R_index_pip_joint multiplier=1.097 offset=0
- joint R_index_pip_joint: limit lower=0 upper=1.5707963267948966 effort=1.764 velocity=0.308 -> lower=0 upper=0.907963267948966 effort=1.764 velocity=0.308
- joint R_middle_dip_joint: mimic joint=R_middle_pip_joint multiplier=0.3 offset=0 -> joint=R_middle_pip_joint multiplier=1.097 offset=0
- joint R_middle_pip_joint: limit lower=0 upper=1.5707963267948966 effort=1.764 velocity=0.308 -> lower=0 upper=1.2707963267948966 effort=1.764 velocity=0.308
- joint R_pinky_dip_joint: mimic joint=R_pinky_pip_joint multiplier=0.3 offset=0 -> joint=R_pinky_pip_joint multiplier=1.097 offset=0
- joint R_ring_dip_joint: mimic joint=R_ring_pip_joint multiplier=0.3 offset=0 -> joint=R_ring_pip_joint multiplier=1.097 offset=0
- joint R_ring_pip_joint: limit lower=0 upper=1.5707963267948966 effort=1.764 velocity=0.308 -> lower=0 upper=1.3707963267948966 effort=1.764 velocity=0.308
- joint R_thumb_dip_joint: mimic joint=R_thumb_mcp_joint multiplier=0.5 offset=0 -> joint=R_thumb_mcp_joint multiplier=1.3 offset=0
- joint R_thumb_pip_joint: mimic joint=R_thumb_mcp_joint multiplier=0.5 offset=0 -> joint=R_thumb_mcp_joint multiplier=1.33 offset=0

File: robots/hands/omnipro_hand/omniprohand_right.urdf (robot description, URDF)
Before this commit: robot omniprohand, 25 links, 24 joints
Joints:
- joint thumb_cmc_yaw: limit lower=0 upper=1.3868 effort=100 velocity=1 -> lower=0 upper=0.3 effort=100 velocity=1
- joint thumb_ip: limit lower=0 upper=0.3781 effort=100 velocity=1 -> lower=0 upper=1.3781 effort=100 velocity=1
- joint thumb_mcp: limit lower=0 upper=0.2908 effort=100 velocity=1 -> lower=0 upper=1.2908 effort=100 velocity=1
